File: DumbWatch_PCB/DumbWatch_PCB.kicad_sch (KiCad schematic)
At the start: 0 parts

Commit message: update PCB, edit fp-lib-table to have relative path with /..., add external models for footprints - models - and symbols
Parts:
- added DS1: NHD-C12832A1Z-FSW-FBW-3V3, WatchParts:LCD_NHD-C12832A1Z-FSW-FBW-3V3, symbol WatchParts:NHD-C12832A1Z-FSW-FBW-3V3
- added U1: XIAO-ESP32-C5-SMD, WatchParts:XIAO-ESP32-C5-SMD, symbol WatchParts:XIAO-ESP32-C5-SMD
